File: kicad_proj/assembly_line_enviro_tester/assembly_line_enviro_tester.kicad_pcb (KiCad board)
At the start: 4 copper layers, 53 x 35.5 mm, 51 parts, among them J1 Conn_01x02_Female, J2 0524353071, J3 Tag_Connect_6_Pin, Q1 MMSS8050-L-TP, Q2 MMSS8050-L-TP, Q3 2N7002-TP, Q4 INL-5APT30, U1 ESP32-WROOM-32D, U2 TPS56339DDCR, U3 HDC1080DMBR

Commit message: first layout try
Parts:
- added SW1: PTS_647_SN70_SMTR2_LFS, lib_fp:PTS_647_SN70_SMTR2_LFS, F.Cu at (20.5, -73.2)
- added TP2: TestPoint, TestPoint:TestPoint_Plated_Hole_D2.0mm, F.Cu at (22.6, -67.1)
- added TP3: TestPoint, TestPoint:TestPoint_Plated_Hole_D2.0mm, F.Cu at (22.6, -62.2)
- added TP4: TestPoint, TestPoint:TestPoint_Plated_Hole_D2.0mm, F.Cu at (22.6, -57.0)
- C1, C12, C13, C14, C15, C17, C18, C19, C2, C20, C21, C22, C3, C4, C5, C6, C8, C9: footprint lib_fp:CHIP_0603N -> Capacitor_SMD:C_0603_1608Metric
- C10, C11, C7: footprint lib_fp:CHIP_1206N -> Capacitor_SMD:C_1206_3216Metric
- C16: footprint lib_fp:CHIP_0805N -> Capacitor_SMD:C_0805_2012Metric
- F1: footprint footprints:FUSC455X324X155L45N -> Fuse:Fuse_1812_4532Metric_Castellated
- F2: footprint footprints:FUSE_0603N -> Fuse:Fuse_0603_1608Metric
- FB1: footprint lib_fp:CHIP_0805N -> Inductor_SMD:L_0805_2012Metric
- R1: footprint lib_fp:CHIP_1206N -> Resistor_SMD:R_1206_3216Metric
- R10, R11, R2, R3, R4, R5, R6, R7, R8, R9: footprint lib_fp:CHIP_0603N -> Resistor_SMD:R_0603_1608Metric
- moved J1 27.8 mm to (48.0, -79.6), turned to 180 degrees
- moved U3 27.4 mm to (47.8, -49.4)
- moved C20 27.4 mm to (50.7, -48.6)
- moved D1 24.6 mm to (45.9, -74.4), turned to 90 degrees
- moved Q3 24.3 mm to (21.3, -48.6), turned to 270 degrees
- moved F1 20.7 mm to (50.6, -74.5), turned to 90 degrees
- moved Q4 20.5 mm to (42.7, -57.9), turned to 180 degrees
- moved C3 20.2 mm to (48.0, -69.2), turned to 180 degrees
- moved R8 19.8 mm to (33.5, -68.9), turned to 0 degrees
- moved R10 19.8 mm to (39.9, -58.8), turned to 270 degrees
- moved R9 19.7 mm to (20.8, -51.2), turned to 0 degrees
- moved C9 19.5 mm to (42.4, -65.3), turned to 90 degrees
- moved C8 19.5 mm to (43.9, -65.3), turned to 90 degrees
- moved C5 19.4 mm to (48.0, -67.7), turned to 180 degrees
- moved BZ1 19.4 mm to (31.5, -52.7), turned to 180 degrees
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Connections:
- D2 pad 1: /SDA -> /SCL
- D2 pad 2: /SCL -> /SDA
- L1 pad 1: Net-(C3-Pad1) -> +5V
- L1 pad 2: Net-(C3-Pad2) -> GND
- L1 pad 3: GND -> Net-(C3-Pad2)
- L1 pad 4: +5V -> Net-(C3-Pad1)
Routing:
- net GND: track 99.0 -> 173.0 mm, vias 53 -> 13
- net +3V3: track 130.7 -> 71.1 mm, vias 5 -> 4
- net Net-(TP4-Pad1): track 0.00 -> 21.6 mm, vias 0 -> 1
- net /EN: track 35.5 -> 52.2 mm
- net Net-(TP3-Pad1): track 0.00 -> 16.1 mm, vias 0 -> 1
- net Net-(R7-Pad2): track 16.6 -> 3.45 mm
- net /RTS: track 24.2 -> 12.4 mm
- net Net-(TP2-Pad1): track 0.00 -> 10.9 mm, vias 0 -> 1
- net Net-(C15-Pad1): track 4.84 -> 13.0 mm, vias 0 -> 2
- net Net-(Q4-Pad1): track 28.1 -> 34.8 mm, vias 2 -> 1
- net /IO0: track 13.2 -> 7.77 mm, vias 2 -> 0
- net +5V: track 49.6 -> 44.6 mm, vias 6 -> 2
- net /SCL: track 64.5 -> 69.3 mm, vias 4 -> 5
- net Net-(C3-Pad1): track 18.4 -> 13.5 mm
- net Net-(C19-Pad1): track 11.0 -> 7.02 mm
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- added copper zone on In2.Cu, net +3V3
- removed copper zone on In2.Cu, net GND
Other:
- outline, holes or cut-outs redrawn
- net class Default: clearance 0.15 -> 0.2; trace_width 0.15 -> 0.25
- net class Power added: clearance 0.2, trace_width 0.3, via_dia 0.6, via_drill 0.3
- rule solder_mask_min_width: 0.25 -> 0.1
- rule trace_clearance: 0.15 -> 0.2
