File: kicad_proj/assembly_line_enviro_tester/assembly_line_enviro_tester.sch (KiCad schematic (older format))
At the start: 55 parts, among them J1 Conn_01x02_Female, J2 0524353071, J3 Tag_Connect_6_Pin, Q1 MMSS8050-L-TP, Q2 MMSS8050-L-TP, Q3 2N7002-TP, Q4 INL-5APT30, SW1 PTS_647_SN70_SMTR2_LFS, U1 ESP32-WROOM-32D, U2 TPS56339DDCR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

Commit message: first layout try
Parts:
- BZ1: symbol misc:SMI-1324-TW-5V-3-R -> assembly_line_enviro_tester-rescue:SMI-1324-TW-5V-3-R-misc
- C1, C12, C14, C15, C18, C19, C20, C21, C22, C3, C4, C9: footprint lib_fp:CHIP_0603N -> Capacitor_SMD:C_0603_1608Metric; symbol capacitors:CC0603KRX7R9BB104 -> assembly_line_enviro_tester-rescue:CC0603KRX7R9BB104-capacitors
- C10, C11, C7: footprint lib_fp:CHIP_1206N -> Capacitor_SMD:C_1206_3216Metric; symbol capacitors:CL31A106KPHNNNE -> assembly_line_enviro_tester-rescue:CL31A106KPHNNNE-capacitors
- C13: footprint lib_fp:CHIP_0603N -> Capacitor_SMD:C_0603_1608Metric; symbol capacitors:CL10B102KB8WPNC -> assembly_line_enviro_tester-rescue:CL10B102KB8WPNC-capacitors
- C16: footprint lib_fp:CHIP_0805N -> Capacitor_SMD:C_0805_2012Metric; symbol capacitors:C2012X7S1A226M125AC -> assembly_line_enviro_tester-rescue:C2012X7S1A226M125AC-capacitors
- C17, C5, C6, C8: footprint lib_fp:CHIP_0603N -> Capacitor_SMD:C_0603_1608Metric; symbol capacitors:CC0603KRX5R9BB105 -> assembly_line_enviro_tester-rescue:CC0603KRX5R9BB105-capacitors
- C2: footprint lib_fp:CHIP_0603N -> Capacitor_SMD:C_0603_1608Metric; symbol capacitors:CL10B103KB8NNNC -> assembly_line_enviro_tester-rescue:CL10B103KB8NNNC-capacitors
- D1: symbol diodes:P6SMB6.8A-E3_5B -> assembly_line_enviro_tester-rescue:P6SMB6.8A-E3_5B-diodes
- D2: symbol diodes:RCLAMP0582BQTCT -> assembly_line_enviro_tester-rescue:RCLAMP0582BQTCT-diodes
- F1: footprint footprints:FUSC455X324X155L45N -> Fuse:Fuse_1812_4532Metric_Castellated; symbol fuses:0ZCG0150BF2C -> assembly_line_enviro_tester-rescue:0ZCG0150BF2C-fuses
- F2: footprint footprints:FUSE_0603N -> Fuse:Fuse_0603_1608Metric; symbol fuses:0686F2000-01 -> assembly_line_enviro_tester-rescue:0686F2000-01-fuses
- FB1: footprint lib_fp:CHIP_0805N -> Inductor_SMD:L_0805_2012Metric; symbol inductors:742792040 -> assembly_line_enviro_tester-rescue:742792040-inductors
- J2: symbol connectors:0524353071 -> assembly_line_enviro_tester-rescue:0524353071-connectors
- J3: symbol connectors:Tag_Connect_6_Pin -> assembly_line_enviro_tester-rescue:Tag_Connect_6_Pin-connectors
- L1: symbol inductors:ACM4520V-142-2P-T00 -> assembly_line_enviro_tester-rescue:ACM4520V-142-2P-T00-inductors
- L2: symbol inductors:CIGW252010EH4R7MNE -> assembly_line_enviro_tester-rescue:CIGW252010EH4R7MNE-inductors
- Q1, Q2: symbol transistors:MMSS8050-L-TP -> assembly_line_enviro_tester-rescue:MMSS8050-L-TP-transistors
- Q3: symbol mosfets:2N7002-TP -> assembly_line_enviro_tester-rescue:2N7002-TP-mosfets
- Q4: symbol transistors:INL-5APT30 -> assembly_line_enviro_tester-rescue:INL-5APT30-transistors
- R1: footprint lib_fp:CHIP_1206N -> Resistor_SMD:R_1206_3216Metric; symbol resistors:SR732BTTD1R00D -> assembly_line_enviro_tester-rescue:SR732BTTD1R00D-resistors
- R10: footprint lib_fp:CHIP_0603N -> Resistor_SMD:R_0603_1608Metric; symbol resistors:RC0603JR-07220RL -> assembly_line_enviro_tester-rescue:RC0603JR-07220RL-resistors
- R11, R6, R9: footprint lib_fp:CHIP_0603N -> Resistor_SMD:R_0603_1608Metric; symbol resistors:RC0603JR-0730RL -> assembly_line_enviro_tester-rescue:RC0603JR-0730RL-resistors
- R2, R3, R8: footprint lib_fp:CHIP_0603N -> Resistor_SMD:R_0603_1608Metric; symbol resistors:RC0603JR-0710KL -> assembly_line_enviro_tester-rescue:RC0603JR-0710KL-resistors
- R4, R5: footprint lib_fp:CHIP_0603N -> Resistor_SMD:R_0603_1608Metric; symbol resistors:RC0603JR-074K7L -> assembly_line_enviro_tester-rescue:RC0603JR-074K7L-resistors
- R7: footprint lib_fp:CHIP_0603N -> Resistor_SMD:R_0603_1608Metric; symbol resistors:RC0603FR-0730K9L -> assembly_line_enviro_tester-rescue:RC0603FR-0730K9L-resistors
- SW1: symbol misc:PTS_647_SN70_SMTR2_LFS -> assembly_line_enviro_tester-rescue:PTS_647_SN70_SMTR2_LFS-misc
- U1: symbol ics:ESP32-WROOM-32D -> assembly_line_enviro_tester-rescue:ESP32-WROOM-32D-ics
- U2: symbol ics:TPS56339DDCR -> assembly_line_enviro_tester-rescue:TPS56339DDCR-ics
- U3: symbol ics:HDC1080DMBR -> assembly_line_enviro_tester-rescue:HDC1080DMBR-ics
Connections:
- net +5V: now also L1.1; no longer L1.4
- net GND: now also L1.2; no longer L1.3
- net SCL: now also D2.1 (A1); no longer D2.2 (A2)
- net SDA: now also D2.2 (A2); no longer D2.1 (A1)
- net at C3.2, C5.2, D1.A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: now also L1.3; no longer L1.2
- net at C3.1, C5.1, D1.C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: now also L1.4; no longer L1.1
